File: HW/PWM_DAC/Power.kicad_sch (KiCad schematic)
At the start: 38 parts, among them J501 1715721, Q501 SI5618A, Q502 MMBT3904, U10 TBA2-2423, U19 TPS7A3901DSCR, U21 TPS7A3901DSCR

Commit message: Schematic done
Parts:
- added D6: APFA3010LSEEZGKQBKC, LED_SMD:LED_Kingbright_APFA3010_3x1.5mm_Horizontal, symbol LED:APFA3010
- added D7: MMSZ5240C-HE3_A-08, Diode_SMD:D_SOD-123, symbol Diode:DZ2S100X0L
- added R42, R43: 2k67/1%/250mW, Resistor_SMD:R_0805_2012Metric_Pad1.20x1.40mm_HandSolder, symbol Device:R
- added TP10, TP9: TestPoint, TestPoint:TestPoint_Pad_D1.5mm, symbol Connector:TestPoint
- C37: footprint (none) -> Capacitor_SMD:C_1206_3216Metric_Pad1.33x1.80mm_HandSolder
- C38: renamed from C36; footprint (none) -> Capacitor_SMD:C_0603_1608Metric_Pad1.08x0.95mm_HandSolder
- C40: renamed from C32; footprint (none) -> Capacitor_SMD:C_0603_1608Metric_Pad1.08x0.95mm_HandSolder
- C41: renamed from C33; footprint (none) -> Capacitor_SMD:C_0603_1608Metric_Pad1.08x0.95mm_HandSolder
- C42: renamed from C34; footprint (none) -> Capacitor_SMD:C_1206_3216Metric_Pad1.33x1.80mm_HandSolder
- C43: renamed from C35; footprint (none) -> Capacitor_SMD:C_1206_3216Metric_Pad1.33x1.80mm_HandSolder
- D2: renamed from D502; footprint Diode_SMD:D_SOD-123 -> Diode_SMD:D_SOD-123F
- R32: renamed from R37; value xx/1%/100mW -> 10k/1%/100mW
- R33: renamed from R38; value 140k/1%/100mW -> 100k/1%/100mW
- R34: renamed from R501; value 100k -> 100k/1%/100mW
- R35: renamed from R39; value 160k/1%/100mW -> 90k9/1%/100mW
- R36: renamed from R40; value xx/1%/100mW -> 10k/1%/100mW
- R37: renamed from R502; value 100k -> 100k/1%/100mW
- R38: renamed from R46; value xx/1%/100mW -> 10k/1%/100mW
- R39: renamed from R47; value 105k/1%/100mW -> 42k2/1%/100mW
- R40: renamed from R51; value 107k/1%/100mW -> 32k4/1%/100mW
- R41: renamed from R52; value xx/1%/100mW -> 10k/1%/100mW
- renumbered C77 to C32, C79 to C33, C80 to C34, C82 to C35, C83 to C36, C86 to C39, C95 to C44, C96 to C45, C99 to C46, C100 to C47, D501 to D1, J501 to J1, Q501 to Q2, Q502 to Q3, TP28 to TP5, TP29 to TP6, TP34 to TP7, TP37 to TP8, U19 to U10, U21 to U11, U10 to U12
Connections:
- net +24V: now also D6.2 (A), TP10.1
- net GND: now also C40.1, C41.2; no longer C37.1, C38.1, J1.2 (Pin_2), R34.2, R37.2, U12.2 (-Vin)
- new net: R42.2, R43.1
- new net: D7.2 (A), R42.1
- new net: D6.1 (R), D7.1 (K)
- new net GND1: C37.1, C38.1, J1.2 (Pin_2), R34.2, R37.2, R43.2, TP9.1, U12.2 (-Vin)
- no-connect marks 0 -> 2
Other:
- moved on the sheet: D1, D2, J1, Q2, Q3, R34, R37

Commit message: Layout done
Parts:
- removed D1: BZX84C10LT1G, Package_TO_SOT_SMD:SOT-23, symbol Diode:BZX84Cxx
- removed D2: 1N4148W, Diode_SMD:D_SOD-123F, symbol Diode:1N4148W
- removed Q2: SI5618A, Package_TO_SOT_SMD:SOT-23, symbol Device:Q_PMOS_GSD
- removed Q3: MMBT3904, Package_TO_SOT_SMD:SOT-23, symbol Transistor_BJT:MMBT3904
- removed R34, R37: 100k/1%/100mW, Resistor_SMD:R_0603_1608Metric_Pad0.98x0.95mm_HandSolder, symbol Device:R
- added D1: MMSZ5240C-HE3_A-08, Diode_SMD:D_SOD-123, symbol Diode:DZ2S100X0L
- added Q2: CSD18501Q5A, Package_TO_SOT_SMD:TDSON-8-1, symbol Transistor_FET:CSD18501Q5A
- added R32: 100k/1%/100mW, Resistor_SMD:R_0603_1608Metric_Pad0.98x0.95mm_HandSolder, symbol Device:R
- added TP21, TP22, TP23: TestPoint, TestPoint:TestPoint_Pad_D1.5mm, symbol Connector:TestPoint
- C33, C34, C44, C45: value 4u7/50V/X7R -> 4.7uF/50V/X7R
- C35, C36, C46, C47: value 10u/35V/X7R -> 10uF/35V/X7R
- R35: value 90k9/1%/100mW -> 90.9k/1%/100mW
- R37: renamed from R42; value 2k67/1%/250mW -> 2.67k/1%/250mW
- R38: renamed from R43; value 2k67/1%/250mW -> 2.67k/1%/250mW
- R40: renamed from R39; value 42k2/1%/100mW -> 42.2k/1%/100mW
- R41: renamed from R40; value 32k4/1%/100mW -> 32.4k/1%/100mW
- renumbered D7 to D2, D6 to D3, R32 to R33, R33 to R34, R38 to R39, R41 to R42, TP5 to TP15, TP6 to TP16, TP10 to TP17, TP9 to TP18, TP7 to TP19, TP8 to TP20
Connections:
- net +15V: now also TP21.1
- net +24V: now also J1.1 (Pin_1), R32.1
- net -15V: now also TP22.1
- net GND: now also TP23.1
- net GND1: now also D1.2 (A), Q2.1 (S), Q2.2 (S), Q2.3 (S); no longer J1.2 (Pin_2)
- new net: D1.1 (K), Q2.4 (G), R32.2
- new net: J1.2 (Pin_2), Q2.5 (D)
Other:
- moved on the sheet: C35, C36, C46, C47, J1
