File: HW/PWM_DAC/DAC.kicad_sch (KiCad schematic)
At the start: 57 parts, among them U3 ADA4522-2, U4 ADA4522-2, U5 ADA4522-2, U6 ADA4522-2, U7 ADA4522-2, U8 MAX4053AEEE+T, U9 MAX4053AEEE+T

Commit message: Schematic done
Parts:
- added TP18, TP19: TestPoint, TestPoint:TestPoint_Pad_D1.5mm, symbol Connector:TestPoint
- C1: renamed from C13; footprint (none) -> Capacitor_SMD:C_0603_1608Metric_Pad1.08x0.95mm_HandSolder
- C10: renamed from C15; value 1uF/50V/X7R -> 1uF/25V/X7R; footprint (none) -> Capacitor_SMD:C_0603_1608Metric_Pad1.08x0.95mm_HandSolder
- C11: renamed from C29; footprint (none) -> Capacitor_SMD:C_0603_1608Metric_Pad1.08x0.95mm_HandSolder
- C12: renamed from C21; footprint (none) -> Capacitor_SMD:C_0603_1608Metric_Pad1.08x0.95mm_HandSolder
- C13: renamed from C6; footprint (none) -> Capacitor_SMD:C_0603_1608Metric_Pad1.08x0.95mm_HandSolder
- C14: renamed from C16; footprint (none) -> Capacitor_SMD:C_0603_1608Metric_Pad1.08x0.95mm_HandSolder
- C15: renamed from C8; value 10uF/16V/X7R -> 10uF/35V/X7R; footprint (none) -> Capacitor_SMD:C_1206_3216Metric_Pad1.33x1.80mm_HandSolder
- C16: renamed from C17; value 10uF/16V/X7R -> 10uF/35V/X7R; footprint (none) -> Capacitor_SMD:C_1206_3216Metric_Pad1.33x1.80mm_HandSolder
- C17: renamed from C30; footprint (none) -> Capacitor_SMD:C_0603_1608Metric_Pad1.08x0.95mm_HandSolder
- C18: renamed from C24; footprint (none) -> Capacitor_SMD:C_0603_1608Metric_Pad1.08x0.95mm_HandSolder
- C19: renamed from C9; value 10uF/16V/X7R -> 10uF/35V/X7R; footprint (none) -> Capacitor_SMD:C_1206_3216Metric_Pad1.33x1.80mm_HandSolder
- C2: renamed from C11; footprint (none) -> Capacitor_SMD:C_0603_1608Metric_Pad1.08x0.95mm_HandSolder
- C20: renamed from C18; value 10uF/16V/X7R -> 10uF/35V/X7R; footprint (none) -> Capacitor_SMD:C_1206_3216Metric_Pad1.33x1.80mm_HandSolder
- C21: renamed from C31; footprint (none) -> Capacitor_SMD:C_0603_1608Metric_Pad1.08x0.95mm_HandSolder
- C22: renamed from C25; footprint (none) -> Capacitor_SMD:C_0603_1608Metric_Pad1.08x0.95mm_HandSolder
- C23: renamed from C10; value 10uF/16V/X7R -> 10uF/35V/X7R; footprint (none) -> Capacitor_SMD:C_1206_3216Metric_Pad1.33x1.80mm_HandSolder
- C24: renamed from C19; value 10uF/16V/X7R -> 10uF/35V/X7R; footprint (none) -> Capacitor_SMD:C_1206_3216Metric_Pad1.33x1.80mm_HandSolder
- C25: renamed from C22; footprint (none) -> Capacitor_SMD:C_0603_1608Metric_Pad1.08x0.95mm_HandSolder
- C26: renamed from C23; footprint (none) -> Capacitor_SMD:C_0603_1608Metric_Pad1.08x0.95mm_HandSolder
- C3: renamed from C14; footprint (none) -> Capacitor_SMD:C_0603_1608Metric_Pad1.08x0.95mm_HandSolder
- C4: renamed from C12; footprint (none) -> Capacitor_SMD:C_0603_1608Metric_Pad1.08x0.95mm_HandSolder
- C5: renamed from C26; value 1uF/50V/X7R -> 1uF/25V/X7R; footprint (none) -> Capacitor_SMD:C_0603_1608Metric_Pad1.08x0.95mm_HandSolder
- C6: renamed from C27; value 1uF/50V/X7R -> 1uF/25V/X7R; footprint (none) -> Capacitor_SMD:C_0603_1608Metric_Pad1.08x0.95mm_HandSolder
- C7: renamed from C28; footprint (none) -> Capacitor_SMD:C_0603_1608Metric_Pad1.08x0.95mm_HandSolder
- C8: renamed from C20; footprint (none) -> Capacitor_SMD:C_0603_1608Metric_Pad1.08x0.95mm_HandSolder
- C9: renamed from C7; value 1uF/50V/X7R -> 1uF/25V/X7R; footprint (none) -> Capacitor_SMD:C_0603_1608Metric_Pad1.08x0.95mm_HandSolder
- R1: renamed from R30; footprint (none) -> Resistor_SMD:R_0603_1608Metric_Pad0.98x0.95mm_HandSolder
- R10: renamed from R6; footprint (none) -> Resistor_SMD:R_0603_1608Metric_Pad0.98x0.95mm_HandSolder
- R11: renamed from R7; footprint (none) -> Resistor_SMD:R_0805_2012Metric_Pad1.20x1.40mm_HandSolder
- R12: renamed from R10; footprint (none) -> Resistor_SMD:R_0805_2012Metric_Pad1.20x1.40mm_HandSolder
- R13: renamed from R8; footprint (none) -> Resistor_SMD:R_0805_2012Metric_Pad1.20x1.40mm_HandSolder
- R14: renamed from R9; footprint (none) -> Resistor_SMD:R_0805_2012Metric_Pad1.20x1.40mm_HandSolder
- R15: renamed from R11; footprint (none) -> Resistor_SMD:R_0805_2012Metric_Pad1.20x1.40mm_HandSolder
- R16: renamed from R12; footprint (none) -> Resistor_SMD:R_0805_2012Metric_Pad1.20x1.40mm_HandSolder
- R17: renamed from R13; footprint (none) -> Resistor_SMD:R_0805_2012Metric_Pad1.20x1.40mm_HandSolder
- R18: renamed from R14; footprint (none) -> Resistor_SMD:R_0805_2012Metric_Pad1.20x1.40mm_HandSolder
- R19: renamed from R16; footprint (none) -> Resistor_SMD:R_0805_2012Metric_Pad1.20x1.40mm_HandSolder
- R2: renamed from R29; footprint (none) -> Resistor_SMD:R_0603_1608Metric_Pad0.98x0.95mm_HandSolder
- R20: renamed from R15; footprint (none) -> Resistor_SMD:R_0805_2012Metric_Pad1.20x1.40mm_HandSolder
- R3: renamed from R25; footprint (none) -> Resistor_SMD:R_0603_1608Metric_Pad0.98x0.95mm_HandSolder
- R4: renamed from R27; footprint (none) -> Resistor_SMD:R_0603_1608Metric_Pad0.98x0.95mm_HandSolder
- R5: renamed from R26; footprint (none) -> Resistor_SMD:R_0603_1608Metric_Pad0.98x0.95mm_HandSolder
- R6: renamed from R28; footprint (none) -> Resistor_SMD:R_0603_1608Metric_Pad0.98x0.95mm_HandSolder
- R7: renamed from R3; footprint (none) -> Resistor_SMD:R_0603_1608Metric_Pad0.98x0.95mm_HandSolder
- R8: renamed from R5; footprint (none) -> Resistor_SMD:R_0603_1608Metric_Pad0.98x0.95mm_HandSolder
- R9: renamed from R4; footprint (none) -> Resistor_SMD:R_0603_1608Metric_Pad0.98x0.95mm_HandSolder
- TP1: renamed from TP3; footprint (none) -> TestPoint:TestPoint_Pad_D1.5mm
- TP2: renamed from TP4; footprint (none) -> TestPoint:TestPoint_Pad_D1.5mm
- TP3: renamed from TP1; footprint (none) -> TestPoint:TestPoint_Pad_D1.5mm
- TP4: renamed from TP2; footprint (none) -> TestPoint:TestPoint_Pad_D1.5mm
- U1: renamed from U4; value ADA4522-2 -> ADA4522-2ARZ-RL; footprint (none) -> Package_SO:SOIC-8_3.9x4.9mm_P1.27mm
- U2: renamed from U3; value ADA4522-2 -> ADA4522-2ARZ-RL; footprint (none) -> Package_SO:SOIC-8_3.9x4.9mm_P1.27mm
- U5: value ADA4522-2 -> ADA4522-2ARZ-RL; footprint (none) -> Package_SO:SOIC-8_3.9x4.9mm_P1.27mm
- U6: renamed from U7; value ADA4522-2 -> ADA4522-2ARZ-RL; footprint (none) -> Package_SO:SOIC-8_3.9x4.9mm_P1.27mm
- U7: renamed from U6; value ADA4522-2 -> ADA4522-2ARZ-RL; footprint (none) -> Package_SO:SOIC-8_3.9x4.9mm_P1.27mm
- renumbered U8 to U3, U9 to U4
Connections:
- net at R16.1, U7.6 (-), U7.7: now also TP19.1
- net at R15.1, U1.1, U1.2 (-): now also TP18.1
Other:
- moved on the sheet: C1, C11, C2, C21, C3, C4, U1C, U2C, U5C, U6C, U7C

Commit message: Layout done
Parts:
- added TP10, TP5, TP6, TP9: TestPoint, TestPoint:TestPoint_Pad_D1.5mm, symbol Connector:TestPoint
- R7, R8: value 88k7/1%/100mW -> 88.7k/1%/100mW
- TP1, TP2, TP3, TP4: now left out of the parts list
- U3, U4: footprint Package_SO:SSOP-16_3.9x4.9mm_P0.635mm -> Package_SO:QSOP-16_3.9x4.9mm_P0.635mm
- renumbered TP18 to TP7, TP19 to TP8
Connections:
- net at R17.2, R18.1, U6.1: now also TP10.1
- net at C15.2, C19.2, C23.2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: now also TP5.1
- net at C16.2, C20.2, C24.2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: now also TP6.1
- net at R15.2, R16.2, R17.1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: now also TP9.1
Other:
- moved on the sheet: C1, C11, C12, C17, C18, C2, C21, C22, C25, C26, C3, C4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

Commit message: PCB files send
Parts:
- R1, R2: now not fitted; now left out of the parts list
Changed lines of the file:
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@@
 		(body_style 1)
 		(exclude_from_sim no)
-		(in_bom yes)
+		(in_bom no)
 		(on_board yes)
 		(in_pos_files yes)
-		(dnp no)
+		(dnp yes)
 		(property "Reference" "R1"
 			(at 26.67 59.944 90)
@@
 		(body_style 1)
 		(exclude_from_sim no)
-		(in_bom yes)
+		(in_bom no)
 		(on_board yes)
 		(in_pos_files yes)
-		(dnp no)
+		(dnp yes)
 		(property "Reference" "R2"
 			(at 26.162 150.114 90)
