File: HW/PWM_DAC/PWM_DAC.kicad_pcb (KiCad board)
At the start: 4 copper layers, 61 x 61 mm, 134 parts, among them J1 1715721, J2 1715721, J3 PMOD, Q1 2N7002, Q2 SI5618A, Q3 MMBT3904, U1 ADA4522-2ARZ-RL, U10 TPS7A3901DSCR, U11 TPS7A3901DSCR, U12 TBA2-2423, U2 ADA4522-2ARZ-RL, U3 MAX4053AEEE+T, U4 MAX4053AEEE+T, U5 ADA4522-2ARZ-RL, U6 ADA4522-2ARZ-RL, U7 ADA4522-2ARZ-RL, U8 ADA4522-2ARZ-RL, U9 ADR4550

Commit message: Layout done
Parts:
- removed the D2 at (172.7, 83.1)
- removed Q3: MMBT3904, Package_TO_SOT_SMD:SOT-23
- removed the R34 at (175.5, 90.7)
- removed the R37 at (175.5, 86.5)
- added R32: 100k/1%/100mW, Resistor_SMD:R_0603_1608Metric_Pad0.98x0.95mm_HandSolder, F.Cu at (174.0, 90.9)
- added TP10: TestPoint, TestPoint:TestPoint_Pad_D1.5mm, F.Cu at (143.9, 132.7)
- added TP21: TestPoint, TestPoint:TestPoint_Pad_D1.5mm, F.Cu at (140.9, 81.4)
- added TP22: TestPoint, TestPoint:TestPoint_Pad_D1.5mm, F.Cu at (134.5, 81.4)
- added TP23: TestPoint, TestPoint:TestPoint_Pad_D1.5mm, F.Cu at (149.9, 93.3)
- added TP5: TestPoint, TestPoint:TestPoint_Pad_D1.5mm, F.Cu at (157.3, 121.9)
- added TP6: TestPoint, TestPoint:TestPoint_Pad_D1.5mm, F.Cu at (156.3, 137.9)
- added TP9: TestPoint, TestPoint:TestPoint_Pad_D1.5mm, F.Cu at (142.1, 123.5)
- C33, C34, C44, C45: value 4u7/50V/X7R -> 4.7uF/50V/X7R
- C35, C36, C46, C47: value 10u/35V/X7R -> 10uF/35V/X7R
- D1: value BZX84C10LT1G -> MMSZ5240C-HE3_A-08; footprint Package_TO_SOT_SMD:SOT-23 -> Diode_SMD:D_SOD-123
- Q2: value SI5618A -> CSD18501Q5A; footprint Package_TO_SOT_SMD:SOT-23 -> Package_TO_SOT_SMD:TDSON-8-1
- R29, R30: value 0R4/1%/100mW -> 0.4R/1%/100mW
- R31: value 4R99/0.1%/100mW -> 4.99R/0.1%/100mW
- R35: value 90k9/1%/100mW -> 90.9k/1%/100mW
- R37: renamed from R42; value 2k67/1%/250mW -> 2.67k/1%/250mW
- R38: renamed from R43; value 2k67/1%/250mW -> 2.67k/1%/250mW
- R40: renamed from R39; value 42k2/1%/100mW -> 42.2k/1%/100mW
- R41: renamed from R40; value 32k4/1%/100mW -> 32.4k/1%/100mW
- R7, R8: value 88k7/1%/100mW -> 88.7k/1%/100mW
- U3, U4: footprint Package_SO:SSOP-16_3.9x4.9mm_P0.635mm -> Package_SO:QSOP-16_3.9x4.9mm_P0.635mm
- U9: value ADR4550 -> ADR4550BRZ-R7
- moved FID1 76.3 mm to (185.9, 133.8)
- moved TP25 11.7 mm to (179.1, 132.4)
- moved Q2 8.51 mm to (173.8, 83.7), turned to 90 degrees
- moved R1 5.85 mm to (173.9, 114.9), turned to 180 degrees
- moved R2 5.82 mm to (173.9, 131.1), turned to 180 degrees
- moved D1 3.54 mm to (176.2, 90.2)
- moved R5 3.41 mm to (174.8, 110.5)
- moved R6 3.41 mm to (174.8, 126.6)
- moved TP15 2.41 mm to (144.8, 94.7)
- moved FID2 1.57 mm to (185.1, 106.1)
- moved C32 1.41 mm to (137.7, 85.7), turned to 90 degrees
- moved C5 1.27 mm to (173.9, 113.0), turned to 0 degrees
- moved TP13 1.26 mm to (166.8, 122.6)
- moved C6 1.26 mm to (173.9, 129.1), turned to 0 degrees
- moved TP7 1.13 mm to (144.5, 110.0)
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- renumbered D7 to D2, D6 to D3, R32 to R33, R33 to R34, R38 to R39, R41 to R42, TP12 to TP11, TP11 to TP12, TP5 to TP15, TP6 to TP16, TP10 to TP17, TP9 to TP18, TP7 to TP19, TP8 to TP20, TP15 to TP24, TP16 to TP25, TP17 to TP26, TP18 to TP7, TP19 to TP8
Connections:
- D1 pad 1: Net-(D1-A) -> Net-(D1-K)
- D1 pad 2: unconnected-(D1-NC-Pad2) -> GND1
- J1 pad 1: Net-(J1-Pin_1) -> +24V
- J1 pad 2: GND1 -> Net-(J1-Pin_2)
- Q2 pad 1: Net-(D1-A) -> GND1
- Q2 pad 2: +24V -> GND1
- Q2 pad 3: Net-(J1-Pin_1) -> GND1
Routing:
- net VEE: track 0.00 -> 103.1 mm, vias 0 -> 9
- net -5V: track 0.00 -> 63.6 mm, vias 0 -> 4
- net +5V: track 0.00 -> 56.5 mm, vias 0 -> 4
- net /DAC/VREF_P: track 0.00 -> 34.7 mm
- net /DAC/CLK: track 0.00 -> 32.6 mm
- net /DAC/VREF_N: track 0.00 -> 32.3 mm
- net Net-(U7B--): track 0.00 -> 28.4 mm
- net VCC: track 0.00 -> 23.6 mm, vias 0 -> 12
- net /DAC/X1B: track 0.00 -> 23.5 mm
- net /CONN_IN/PWM_F: track 0.00 -> 22.6 mm
- net /DAC/X1A: track 0.00 -> 20.5 mm, vias 0 -> 2
- net Net-(U6A--): track 0.00 -> 19.0 mm
- net Net-(U7A-+): track 0.00 -> 17.9 mm
- net /CONN_OUT/DAC_OUT: track 0.00 -> 17.0 mm
- net Net-(U1A-+): track 0.00 -> 16.4 mm
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- added copper zone on F.Cu, net +15V
- added copper zone on In2.Cu, net +15V
- added copper zone on F.Cu, net +24V
- added copper zone on In2.Cu, net +24V
- added copper zone on F.Cu, net +5V
- added copper zone on In2.Cu, net +5V
- added copper zone on F.Cu, net +5VL
- added copper zone on F.Cu, net -15V
- added copper zone on In2.Cu, net -15V
- added copper zone on F.Cu, net -5V
- added copper zone on B.Cu, net GND
- added copper zone on F.Cu, net GND
- added copper zone on In1.Cu, net GND
- added copper zone on In2.Cu, net GND
- added copper zone on B.Cu, net GND1
- added copper zone on F.Cu, net GND1
- added copper zone on In1.Cu, net GND1
- added copper zone on B.Cu, net Net-(J1-Pin_2)
- added copper zone on F.Cu, net Net-(J1-Pin_2)
- added copper zone on In1.Cu, net Net-(J1-Pin_2)
- added copper zone on In2.Cu, net Net-(J1-Pin_2)
- added copper zone on F.Cu, net VCC
- added copper zone on In2.Cu, net VCC
- added copper zone on F.Cu, net VEE
- added copper zone on In2.Cu, net VEE

Commit message: Layout
Parts:
- moved TP25 0.50 mm to (179.1, 132.9)
- moved TP4 0.40 mm to (165.8, 125.4)
Routing:
- net VCC: track 23.6 -> 170.2 mm
- net -5V: track 63.6 -> 111.5 mm
- net +5V: track 56.5 -> 64.3 mm
- net VEE: track 103.1 -> 99.1 mm
- net /DAC/X0B: track 15.4 -> 17.1 mm
- net Net-(U4-Y1): track 2.69 -> 1.79 mm
- net GND: vias 82 -> 95
- added copper zone on In2.Cu, net -5V

Commit message: PCB files send
Parts:
- U9: value ADR4550BRZ-R7 -> LT1461CCS8-5#TRPBF
Routing:
- net -5V: track 111.5 -> 117.2 mm
- net Net-(U2A--): track 12.0 -> 13.1 mm
- net GND1: vias 10 -> 13
- net GND: vias 95 -> 106
Other:
- board text added: "OUTPUT"
